Commit message: Edit Rviz config file

File: src/ur5_volcani_description/urdf/ur5_volcani.urdf.xacro (robot description, xacro)
@@ -23,5 +23,5 @@
   <!-- Table top at 0.98m height, rotated 180 deg yaw (same as volcaniarm) -->
   <joint name="world_to_base" type="fixed">
-    <origin xyz="0 0 0.98" rpy="0 0 3.14159" />
+    <origin xyz="0 0 0.98" rpy="0 0 0" />
     <parent link="world" />
     <child link="table_top_link" />
